Commit message: new file:   mani_skill/assets/robots/panda/panda_v1.srdf 	modified:   mani_skill/assets/robots/panda/panda_v1.urdf 	modified:   mani_skill/envs/scenes/base_env.py

File: mani_skill/assets/robots/panda/panda_v1.urdf (robot description, URDF)
Before this commit: robot panda, 15 links, 14 joints
Links:
- link panda_hand: geometry collision mesh filename=franka_description/meshes/collision/hand.stl; visual mesh filename=franka_description/meshes/visual/hand.dae
- link panda_leftfinger: geometry collision box size=17.5e-3 15.2e-3 18.5e-3; collision box size=17.5e-3 7e-3 23.5e-3
- link panda_link0: geometry collision mesh filename=franka_description/meshes/collision/link0.stl; visual mesh filename=franka_description/meshes/visual/link0.dae
- link panda_link1: geometry collision mesh filename=franka_description/meshes/collision/link1.stl; visual mesh filename=franka_description/meshes/visual/link1.dae
- link panda_link2: geometry collision mesh filename=franka_description/meshes/collision/link2.stl; visual mesh filename=franka_description/meshes/visual/link2.dae
- link panda_link3: geometry collision mesh filename=franka_description/meshes/collision/link3.stl; visual mesh filename=franka_description/meshes/visual/link3.dae
- link panda_link4: geometry collision mesh filename=franka_description/meshes/collision/link4.stl; visual mesh filename=franka_description/meshes/visual/link4.dae
- link panda_link5: geometry collision mesh filename=franka_description/meshes/collision/link5.stl; visual mesh filename=franka_description/meshes/visual/link5.dae
- link panda_link6: geometry collision mesh filename=franka_description/meshes/collision/link6.stl; visual mesh filename=franka_description/meshes/visual/link6.dae
- link panda_link7: geometry collision mesh filename=franka_description/meshes/collision/link7.stl; visual mesh filename=franka_description/meshes/visual/link7.dae
- link panda_rightfinger: geometry collision box size=17.5e-3 15.2e-3 18.5e-3; collision box size=17.5e-3 7e-3 23.5e-3
