Commit message: modified:   mani_skill/agents/robots/panda/panda.py 	modified:   mani_skill/assets/robots/panda/panda_v2.urdf

File: mani_skill/assets/robots/panda/panda_v2.urdf (robot description, URDF)
Before this commit: robot panda, 15 links, 14 joints
Links:
- added link base_slide_x
- added link base_slide_y
- added link base_slide_z
- added link fixed_base
Joints:
- added joint base_prismatic_x: type prismatic, parent fixed_base, child base_slide_x, origin xyz=0 0 0.01 rpy=0 0 0, axis 1 0 0, limit lower=-10 upper=10 effort=1000 velocity=2
- added joint base_prismatic_y: type prismatic, parent base_slide_x, child base_slide_y, origin xyz=0 0 0 rpy=0 0 0, axis 0 1 0, limit lower=-10 upper=10 effort=1000 velocity=2
- added joint base_prismatic_z: type prismatic, parent base_slide_y, child base_slide_z, origin xyz=0 0 0 rpy=0 0 0, axis 0 0 1, limit lower=0 upper=2 effort=1000 velocity=1
- added joint base_revolute_z: type revolute, parent base_slide_z, child panda_link0, origin xyz=0 0 0 rpy=0 0 0, axis 0 0 1, limit lower=-3.14159 upper=3.14159 effort=1000 velocity=1

Commit message: modified:   mani_skill/agents/robots/panda/panda.py 	modified:   mani_skill/assets/robots/panda/panda_v2.urdf 	modified:   mani_skill/envs/scenes/base_env.py 	modified:   mani_skill/utils/scene_builder/table/scene_builder.py

File: mani_skill/assets/robots/panda/panda_v2.urdf (robot description, URDF)
Before this commit: robot panda, 19 links, 18 joints
Links:
- added link camera_base_link
- added link camera_link; visual mesh filename=realsense2_description/meshes/d415.stl
Joints:
- added joint camera_link_joint: type fixed, parent camera_base_link, child camera_link, origin xyz=0 0.02 0.0115 rpy=0 0 0
- added joint realsense_mount_joint: type revolute, parent panda_link0, child camera_base_link, origin xyz=0 0 1 rpy=0 -1.57079632679489 3.1415926, axis 0 1 0, limit lower=-10 upper=10 effort=1000 velocity=2

Commit message: modified:   mani_skill/agents/robots/panda/panda.py 	modified:   mani_skill/assets/robots/panda/panda_v2.urdf

File: mani_skill/assets/robots/panda/panda_v2.urdf (robot description, URDF)
Before this commit: robot panda, 21 links, 20 joints
Links:
- removed link camera_base_link
- added link camera_base_link0
- added link camera_base_link1
Joints:
- removed joint realsense_mount_joint
- added joint camera_link_joint0: type prismatic, parent panda_link0, child camera_base_link0, origin xyz=0 0 0 rpy=0 0 0, axis 0 0 1, limit lower=0 upper=5 effort=1000 velocity=0
- added joint camera_link_joint1: type revolute, parent camera_base_link0, child camera_base_link1, origin xyz=0 0 0 rpy=0 -1.57079632679489 3.1415926, axis 0 1 0, limit lower=-10 upper=10 effort=1000 velocity=0
- joint base_prismatic_x: limit lower=-10 upper=10 effort=1000 velocity=2 -> lower=-10 upper=10 effort=1000 velocity=0
- joint base_prismatic_y: limit lower=-10 upper=10 effort=1000 velocity=2 -> lower=-10 upper=10 effort=1000 velocity=0
- joint base_prismatic_z: limit lower=0 upper=2 effort=1000 velocity=1 -> lower=0 upper=5 effort=1000 velocity=0
- joint base_revolute_z: limit lower=-3.14159 upper=3.14159 effort=1000 velocity=1 -> lower=-10 upper=10 effort=1000 velocity=0
- joint camera_link_joint: parent camera_base_link -> camera_base_link1

Commit message: modified:   mani_skill/agents/robots/panda/panda.py 	modified:   mani_skill/assets/robots/panda/panda_v2.urdf

File: mani_skill/assets/robots/panda/panda_v2.urdf (robot description, URDF)
Before this commit: robot panda, 22 links, 21 joints
Links:
- added link camera_link_back
- added link camera_link_left
- added link camera_link_right
- added link camera_link_top
- link camera_link: geometry 
Joints:
- added joint camera_link_back_joint: type fixed, parent camera_base_link0, child camera_link_back, origin xyz=0 -0.02 -0.0115 rpy=0 0.45 0
- added joint camera_link_left_joint: type fixed, parent camera_base_link0, child camera_link_left, origin xyz=0 0.02 0.0115 rpy=0 0.45 -1.5707963267948966
- added joint camera_link_right_joint: type fixed, parent camera_base_link0, child camera_link_right, origin xyz=0 -0.02 0.0115 rpy=0 0.45 1.5707963267948966
- added joint camera_link_top_joint: type fixed, parent camera_base_link0, child camera_link_top, origin xyz=0 -0.02 -0.0115 rpy=0 -1.5707963267948966 0
- joint camera_link_joint: axis (none) -> 0 1 0; child camera_link -> camera_base_link1; limit (none) -> lower=-10 upper=10 effort=1000 velocity=0; origin xyz=0 0.02 0.0115 rpy=0 0 0 -> xyz=0 0 0 rpy=0 0.45 3.14159265359; parent camera_base_link1 -> camera_base_link0; type fixed -> revolute
- joint camera_link_joint1: axis 0 1 0 -> (none); child camera_base_link1 -> camera_link; limit lower=-10 upper=10 effort=1000 velocity=0 -> (none); origin xyz=0 0 0 rpy=0 -1.57079632679489 3.1415926 -> xyz=0 0.02 0.0115 rpy=0 0 0; parent camera_base_link0 -> camera_base_link1; type revolute -> fixed

Commit message: modified:   mani_skill/assets/robots/panda/panda_v2.urdf 	modified:   mani_skill/utils/scene_builder/replicacad/scene_builder.py

File: mani_skill/assets/robots/panda/panda_v2.urdf (robot description, URDF)
Before this commit: robot panda, 26 links, 25 joints
Joints:
- joint base_prismatic_x: origin xyz=0 0 0.01 rpy=0 0 0 -> xyz=0 0 0 rpy=0 0 0
